File: kicad/TeensyELS.kicad_pcb (KiCad board)
At the start: 2 copper layers, 96 x 85 mm, 47 parts, among them J1 RJ45_Shielded, J2 Conn_01x04_Pin, J3 Conn_01x04_Pin, J4 Screw_Terminal_01x02, Q1 BSS138, Q2 BSS138, Q3 BSS138, Q4 BSS138, Q5 BSS138, Q6 BSS138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

Commit message: Fixed missing traces
Routing:
- net /PadH2: track 72.1 -> 99.9 mm
- net +3.3V: track 237.7 -> 248.1 mm
- net /Dir: track 55.2 -> 63.1 mm
- net Net-(Q2-D): track 53.9 -> 60.4 mm
Changed lines of the file:
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@@
+	)
+	(segment
+		(start 73.25 72.25)
+		(end 79.75 72.25)
+		(width 0.5)
+		(layer "F.Cu")
+		(net 28)
 	)
 	(segment
@@
 	)
 	(segment
-		(start 38.44 53.7)
-		(end 53.68 53.7)
+		(start 27.74 43)
+		(end 35.24 50.5)
+		(width 0.7)
+		(layer "B.Cu")
+		(net 44)
+	)
+	(segment
+		(start 35.24 50.5)
+		(end 50.48 50.5)
+		(width 0.7)
+		(layer "B.Cu")
+		(net 44)
+	)
+	(segment
+		(start 65.245686 60.10494)
+		(end 67.065686 61.92494)
 		(width 0.7)
 		(layer "B.Cu")
@@
 	)
 	(segment
-		(start 53.68 53.7)
+		(start 58.22 58.24)
+		(end 60.08494 60.10494)
+		(width 0.7)
+		(layer "B.Cu")
+		(net 44)
+	)
+	(segment
+		(start 60.08494 60.10494)
+		(end 65.245686 60.10494)
+		(width 0.7)
+		(layer "B.Cu")
+		(net 44)
+	)
+	(segment
+		(start 50.48 50.5)
 		(end 58.22 58.24)
-		(width 0.7)
-		(layer "B.Cu")
-		(net 44)
-	)
-	(segment
-		(start 27.74 43)
-		(end 38.44 53.7)
 		(width 0.7)
 		(layer "B.Cu")
@@
 	)
 	(segment
+		(start 36.5 54.5)
+		(end 34.275 56.725)
+		(width 0.5)
+		(layer "F.Cu")
+		(net 47)
+	)
+	(segment
 		(start 49.145 44.084422)
 		(end 48 45.229422)
@@
 	)
 	(segment
+		(start 48 58.18)
+		(end 48.06 58.24)
+		(width 0.5)
+		(layer "F.Cu")
+		(net 47)
+	)
+	(segment
+		(start 19.5 87.75)
+		(end 20.8 89.05)
+		(width 0.5)
+		(layer "F.Cu")
+		(net 47)
+	)
+	(segment
+		(start 20.8 76.55)
+		(end 20.8 86.45)
+		(width 0.5)
+		(layer "F.Cu")
+		(net 47)
+	)
+	(segment
+		(start 48 45.229422)
+		(end 48 58.18)
+		(width 0.5)
+		(layer "F.Cu")
+		(net 47)
+	)
+	(segment
+		(start 20.8 89.05)
+		(end 20.8 98.95)
+		(width 0.5)
+		(layer "F.Cu")
+		(net 47)
+	)
+	(segment
+		(start 51.825686 39.06494)
+		(end 49.060024 41.830602)
+		(width 0.5)
+		(layer "F.Cu")
+		(net 47)
+	)
+	(segment
+		(start 39.39 54.5)
+		(end 36.5 54.5)
+		(width 0.5)
+		(layer "F.Cu")
+		(net 47)
+	)
+	(segment
+		(start 49.060024 41.830602)
+		(end 49.145 41.915578)
+		(width 0.5)
+		(layer "F.Cu")
+		(net 47)
+	)
+	(segment
+		(start 20.8 98.95)
+		(end 19.5 100.25)
+		(width 0.5)
+		(layer "F.Cu")
+		(net 47)
+	)
+	(segment
+		(start 49.145 41.915578)
+		(end 49.145 44.084422)
+		(width 0.5)
+		(layer "F.Cu")
+		(net 47)
+	)
+	(segment
+		(start 34.275 60.475)
+		(end 19.5 75.25)
+		(width 0.5)
+		(layer "F.Cu")
+		(net 47)
+	)
+	(segment
 		(start 34.275 56.725)
 		(end 34.275 60.475)
@@
 		(net 47)
 	)
-	(segment
-		(start 48 58.18)
-		(end 48.06 58.24)
-		(width 0.5)
-		(layer "F.Cu")
-		(net 47)
-	)
-	(segment
-		(start 19.5 87.75)
-		(end 20.8 89.05)
-		(width 0.5)
-		(layer "F.Cu")
-		(net 47)
-	)
-	(segment
-		(start 20.8 76.55)
-		(end 20.8 86.45)
-		(width 0.5)
-		(layer "F.Cu")
-		(net 47)
-	)
-	(segment
-		(start 48 45.229422)
-		(end 48 58.18)
-		(width 0.5)
-		(layer "F.Cu")
-		(net 47)
-	)
-	(segment
-		(start 20.8 89.05)
-		(end 20.8 98.95)
-		(width 0.5)
-		(layer "F.Cu")
-		(net 47)
-	)
-	(segment
-		(start 37 54)
-		(end 34.275 56.725)
-		(width 0.5)
-		(layer "F.Cu")
-		(net 47)
-	)
-	(segment
-		(start 34.275 60.475)
-		(end 19.5 75.25)
-		(width 0.5)
-		(layer "F.Cu")
-		(net 47)
-	)
-	(segment
-		(start 51.825686 39.06494)
-		(end 49.060024 41.830602)
-		(width 0.5)
-		(layer "F.Cu")
-		(net 47)
-	)
-	(segment
-		(start 49.060024 41.830602)
-		(end 49.145 41.915578)
-		(width 0.5)
-		(layer "F.Cu")
-		(net 47)
-	)
-	(segment
-		(start 20.8 98.95)
-		(end 19.5 100.25)
-		(width 0.5)
-		(layer "F.Cu")
-		(net 47)
-	)
-	(segment
-		(start 49.145 41.915578)
-		(end 49.145 44.084422)
-		(width 0.5)
-		(layer "F.Cu")
-		(net 47)
-	)
 	(via
-		(at 37 54)
+		(at 39.39 54.5)
 		(size 1.2)
 		(drill 0.7)
@@
 	)
 	(segment
+		(start 39.39 54.5)
+		(end 44.32 54.5)
+		(width 0.5)
+		(layer "B.Cu")
+		(net 47)
+	)
+	(segment
 		(start 26 87.75)
 		(end 19.5 87.75)
@@
 	)
 	(segment
-		(start 37 54)
-		(end 37.5 54.5)
-		(width 0.5)
-		(layer "B.Cu")
-		(net 47)
-	)
-	(segment
 		(start 44.32 54.5)
 		(end 48.06 58.24)
@@
 	)
 	(segment
-		(start 37.5 54.5)
-		(end 44.32 54.5)
-		(width 0.5)
-		(layer "B.Cu")
-		(net 47)
-	)
-	(segment
 		(start 56 73.989949)
 		(end 51.825686 69.815635)
@@
 	)
 	(segment
+		(start 37.9 54.505075)
+		(end 38.955075 53.45)
+		(width 0.5)
+		(layer "B.Cu")
+		(net 48)
+	)
+	(segment
 		(start 19.5 92.25)
 		(end 26 92.25)
@@
 	)
 	(segment
+		(start 54.225 57.155578)
+		(end 54.225 59.525626)
+		(width 0.5)
+		(layer "B.Cu")
+		(net 48)
+	)
+	(segment
+		(start 38.955075 53.45)
+		(end 50.519422 53.45)
+		(width 0.5)
+		(layer "B.Cu")
+		(net 48)
+	)
+	(segment
 		(start 52 92.25)
 		(end 58.5 92.25)
@@
 	)
 	(segment
+		(start 37.9 58.24)
+		(end 37.9 54.505075)
+		(width 0.5)
+		(layer "B.Cu")
+		(net 48)
+	)
+	(segment
+		(start 54.225 59.525626)
+		(end 51.825686 61.92494)
+		(width 0.5)
+		(layer "B.Cu")
+		(net 48)
+	)
+	(segment
 		(start 35.75 92.25)
 		(end 42.25 92.25)
+		(width 0.5)
+		(layer "B.Cu")
+		(net 48)
+	)
+	(segment
+		(start 50.519422 53.45)
+		(end 54.225 57.155578)
 		(width 0.5)
 		(layer "B.Cu")
@@
 		(net 49)
 	)
+	(segment
+		(start 47.07506 61.92494)
+		(end 49.04 59.96)
+		(width 0.5)
+		(layer "B.Cu")
+		(net 49)
+	)
+	(segment
+		(start 51.42 59.96)
+		(end 53.14 58.24)
+		(width 0.5)
+		(layer "B.Cu")
+		(net 49)
+	)
+	(segment
+		(start 49.04 59.96)
+		(end 51.42 59.96)
+		(width 0.5)
+		(layer "B.Cu")
+		(net 49)
+	)
+	(segment
+		(start 46.745686 61.92494)
+		(end 47.07506 61.92494)
+		(width 0.5)
+		(layer "B.Cu")
+		(net 49)
+	)
