File: kicad/LVGL/TeensyELS.kicad_pcb (KiCad board)
At the start: 4 copper layers, 96.6 x 91.3 mm, 56 parts, among them J1 RJ45_Shielded, J2 Conn_01x04_Pin, J3 Conn_01x14_Socket, J4 Screw_Terminal_01x02, J5 Conn_02x03_Odd_Even, Q1 BSS138, Q2 BSS138, Q3 BSS138, Q4 BSS138, Q5 BSS138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

Commit message: Updated fab files
Parts:
- added ?: , , F.Cu at (21.9, 67.1)
- added ?: , , F.Cu at (21.9, 32.9)
- SW1, SW10, SW2, SW3, SW4, SW5, SW6, SW7, SW8, SW9: footprint Button_Switch_THT:SW_TH_Tactile_Omron_B3F-10xx -> Button_Switch_SMD:SW_SPST_Omron_B3FS-101xP
- moved ? 9.02 mm to (20.2, 23.6)
- moved ? 8.81 mm to (110.2, 107.6)
- moved ? 5.84 mm to (110.2, 23.6)
- moved SW1 4.09 mm to (76.5, 77.7)
- moved SW10 4.09 mm to (55.4, 102.6)
- moved SW2 4.09 mm to (22.9, 77.6)
- moved SW3 4.09 mm to (39.1, 77.6)
- moved SW4 4.09 mm to (55.4, 77.6)
- moved SW5 4.09 mm to (22.9, 90.1)
- moved SW6 4.09 mm to (39.1, 90.1)
- moved SW7 4.09 mm to (55.4, 90.1)
- moved SW8 4.09 mm to (22.9, 102.6)
- moved SW9 4.09 mm to (39.1, 102.6)
- moved J5 4.00 mm to (32.5, 24.2), turned to -90 degrees
Connections:
- E1 pad MP: (no net) -> GND
Routing:
- net /Blue: track 54.0 -> 87.0 mm
- net +5V: track 144.9 -> 129.2 mm
- net /UIEncA: track 65.8 -> 79.8 mm
- net /EncA: track 68.8 -> 81.1 mm
- net /UIEncB: track 72.8 -> 83.8 mm
- net /EncB: track 68.5 -> 77.9 mm
- net /BOOT: track 66.0 -> 57.5 mm
- net /Red: track 27.3 -> 19.5 mm, vias 1 -> 2
- net /PadH3: track 97.4 -> 103.5 mm, vias 0 -> 6
- net /PadH1: track 86.6 -> 91.6 mm, vias 0 -> 6
- net /PadH2: track 97.0 -> 101.6 mm, vias 0 -> 6
- net /Green: track 30.6 -> 26.8 mm
- net /PadV1: track 94.1 -> 97.7 mm, vias 1 -> 7
- net GND: track 39.7 -> 42.4 mm, vias 10 -> 11
- net /EN: track 30.1 -> 32.8 mm, vias 0 -> 2
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Other:
- board text removed: "TeensyELS v0.5"
