File: kicad/LVGL/TeensyELS.kicad_sch (KiCad schematic)
At the start: 51 parts, among them J1 RJ45_Shielded, J2 Conn_01x04_Pin, J4 Screw_Terminal_01x02, J5 Conn_02x03_Odd_Even, Q1 BSS138, Q2 BSS138, Q3 BSS138, Q4 BSS138, Q5 BSS138, Q6 BSS138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

Commit message: Updated fab files
Parts:
- added J3: Conn_01x14_Socket, Connector_PinHeader_2.54mm:PinHeader_1x14_P2.54mm_Vertical, symbol Connector:Conn_01x14_Socket
Connections:
- net +3.3V: now also J3.14 (Pin_14), J3.7 (Pin_7)
- net Blue: now also Q9.1 (G)
- net GND: now also E1.MP, J3.13 (Pin_13)
- net Green: no longer Q9.1 (G)
- net LCD_CLK: now also J3.8 (Pin_8)
- net LCD_CS: now also J3.12 (Pin_12)
- net LCD_DC: now also J3.10 (Pin_10)
- net LCD_MOSI: now also J3.9 (Pin_9)
- net LCD_Rst: now also J3.11 (Pin_11)
- new net LCD_MISO: J3.6 (Pin_6)
