File: kicad/LVGL/_autosave-TeensyELS.kicad_sch (KiCad schematic)
At the start: 52 parts, among them J1 RJ45_Shielded, J2 Conn_01x04_Pin, J3 Conn_01x14_Socket, J4 Screw_Terminal_01x02, J5 Conn_02x03_Odd_Even, Q1 BSS138, Q2 BSS138, Q3 BSS138, Q4 BSS138, Q5 BSS138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

Commit message: Updated fab files
Connections:
- net GND: now also E1.MP
Changed lines of the file:
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@@
 (kicad_sch
-	(version 20231120)
+	(version 20250114)
 	(generator "eeschema")
-	(generator_version "8.0")
+	(generator_version "9.0")
 	(paper "A3")
 	(junction
@@
 		(color 0 0 0 0)
 	)
+	(junction
+		(at 277.0589 65.8586)
+		(diameter 0)
+		(color 0 0 0 0)
+	)
 	(wire
 		(pts
@@
 	(wire
 		(pts
-			(xy 311.15 29.21) (xy 309.88 29.21)
+			(xy 311.15 33.02) (xy 313.69 33.02)
 		)
 		(stroke
@@
 	(wire
 		(pts
+			(xy 274.5715 65.8586) (xy 274.5715 64.77)
+		)
+		(stroke
+			(width 0)
+			(type default)
+		)
+	)
+	(wire
+		(pts
 			(xy 285.75 158.75) (xy 285.75 161.29)
 		)
@@
 	(wire
 		(pts
+			(xy 274.5715 64.77) (xy 274.32 64.77)
+		)
+		(stroke
+			(width 0)
+			(type default)
+		)
+	)
+	(wire
+		(pts
 			(xy 284.48 73.66) (xy 284.48 71.3672)
 		)
@@
 	(wire
 		(pts
+			(xy 277.1115 65.8586) (xy 277.0589 65.8586)
+		)
+		(stroke
+			(width 0)
+			(type default)
+		)
+	)
+	(wire
+		(pts
 			(xy 388.62 76.2) (xy 394.97 76.2)
 		)
@@
 	(wire
 		(pts
+			(xy 277.0589 65.8586) (xy 274.5715 65.8586)
+		)
+		(stroke
+			(width 0)
+			(type default)
+		)
+	)
+	(wire
+		(pts
 			(xy 38.1 80.01) (xy 54.61 80.01)
 		)
@@
 		)
 	)
-	(wire
-		(pts
-			(xy 311.15 33.02) (xy 311.15 29.21)
-		)
-		(stroke
-			(width 0)
-			(type default)
-		)
-	)
 	(label "EN"
 		(at 128.27 119.38 180)
@@
 	)
 	(label "Blue"
-		(at 309.88 29.21 0)
+		(at 313.69 33.02 0)
 		(effects
 			(font
@@
 	)
 	(symbol
+		(lib_id "power:GND")
+		(at 274.32 64.77 270)
+		(unit 1)
+		(exclude_from_sim no)
+		(in_bom yes)
+		(on_board yes)
+		(dnp no)
+		(fields_autoplaced yes)
+		(property "Reference" "#PWR041"
+			(at 267.97 64.77 0)
+			(effects
+				(font
+					(size 1.27 1.27)
+				)
+				(hide yes)
+			)
+		)
+		(property "Value" "GND"
+			(at 270.51 64.7699 90)
+			(effects
+				(font
+					(size 1.27 1.27)
+				)
+				(justify right)
+			)
+		)
+		(property "Footprint" ""
+			(at 274.32 64.77 0)
+			(effects
+				(font
+					(size 1.27 1.27)
+				)
+				(hide yes)
+			)
+		)
+		(property "Datasheet" ""
+			(at 274.32 64.77 0)
+			(effects
+				(font
+					(size 1.27 1.27)
+				)
+				(hide yes)
+			)
+		)
+		(property "Description" "Power symbol creates a global label with name \"GND\" , ground"
+			(at 274.32 64.77 0)
+			(effects
+				(font
+					(size 1.27 1.27)
+				)
+				(hide yes)
+			)
+		)
+		(pin "1"
+		)
+		(instances
+			(project "TeensyELS"
+				(path "/b63e3b93-0f97-4c9b-9898-4ea21212bbeb"
+					(reference "#PWR041")
+					(unit 1)
+				)
+			)
+		)
+	)
+	(symbol
 		(lib_id "power:+5V")
 		(at 353.06 198.12 90)
@@
 		(on_board yes)
 		(dnp no)
-		(fields_autoplaced yes)
 		(property "Reference" "R12"
-			(at 273.05 66.04 90)
+			(at 274.32 75.184 90)
 			(effects
 				(font
@@
 		)
 		(property "Value" "10K"
-			(at 273.05 68.58 90)
+			(at 270.002 75.184 90)
 			(effects
 				(font
@@
 		(pin "2"
 		)
+		(pin "MP"
+		)
 		(instances
 			(project ""
@@
 		)
 	)
+	(embedded_fonts no)
 )
